File: hardware/boards/card/v0.1/rythm_card_v0.1.kicad_sch (KiCad schematic)
At the start: 7 parts, among them J1 USB_C_Receptacle, J2 USB_C_Receptacle_USB2.0_16P, U2 STM32H743VGHx

Commit message: testing routing layout on card board
Parts:
- removed H1, H2, H3, H4: MountingHole_Pad, MountingHole:MountingHole_2.2mm_M2_Pad_TopBottom, symbol Mechanical:MountingHole_Pad
- removed J1: USB_C_Receptacle, Connector_USB:USB_C_Receptacle_CNCTech_C-ARA1-AK51X, symbol Connector:USB_C_Receptacle
- removed J2: USB_C_Receptacle_USB2.0_16P, Connector_USB:USB_C_Receptacle_HRO_TYPE-C-31-M-12, symbol Connector:USB_C_Receptacle_USB2.0_16P
- removed U2: STM32H743VGHx, Package_BGA:TFBGA-100_8x8mm_Layout10x10_P0.8mm, symbol MCU_ST_STM32H7:STM32H743VGHx
- added C1, C2, C3: 2.2 uF <100 mΩ ESR, Capacitor_SMD:C_0402_1005Metric, symbol Device:C
- added C15: R, Capacitor_SMD:C_0402_1005Metric, symbol Device:C
- added C16, C17, C18, C19, C28, C29: 4.7uF, Capacitor_SMD:C_0402_1005Metric, symbol Device:C_Small
- added C20, C21, C22, C23, C24, C25, C26, C27, C6: 1uF, Capacitor_SMD:C_0402_1005Metric, symbol Device:C_Small
- added C30: 10nF, Capacitor_SMD:C_0402_1005Metric, symbol Device:C
- added C31, C32: 1uF, Capacitor_SMD:C_0402_1005Metric, symbol Device:C
- added C33: 100nF, Capacitor_SMD:C_0402_1005Metric, symbol Device:C
- added C4: 1uF 600mΩ, Capacitor_SMD:C_0402_1005Metric, symbol Device:C_Small
- added C46, C47: C, symbol Device:C_Small
- added C48, C5, C50, C51, C52, C54, C55, C56, C57, C58, C60, C61, C62, C63, C64, C67, C68: 100nF, Capacitor_SMD:C_0402_1005Metric, symbol Device:C_Small
- added C69: 10uF, Capacitor_SMD:C_0402_1005Metric, symbol Device:C_Small
- added D1: POWER, LED_SMD:LED_0402_1005Metric, symbol Device:LED
- added D2: STATUS, LED_SMD:LED_0402_1005Metric, symbol Device:LED
- added D3: 1N4148WS, Diode_SMD:D_SOD-323, symbol Device:D
- added D4: STATUS2, LED_SMD:LED_0402_1005Metric, symbol Device:LED
- added F1: Polyfuse, Fuse:Fuse_0805_2012Metric, symbol Device:Polyfuse
- added FB1: 120R, Inductor_SMD:L_0805_2012Metric, symbol Device:FerriteBead
- added FB2, FB3, FB4, FB5: 1K @100MHz, Inductor_SMD:L_0603_1608Metric, symbol Device:FerriteBead_Small
- added IC1: NAU88C22YG, Package_DFN_QFN:QFN-32-1EP_5x5mm_P0.5mm_EP3.6x3.6mm, symbol NAU88C22YG:NAU88C22YG
- added IC2: IS42S32160F-6BLI, Package_BGA:BGA-90_8.0x13.0mm_Layout2x3x15_P0.8mm, symbol IS42S32160F-6BLI:IS42S32160F-6BLI
- added Q1: PMV37EN22, Package_TO_SOT_SMD:TSOT-23, symbol Transistor_FET:Q_NMOS_GSD
- added R1, R2: 4.7k, Resistor_SMD:R_0402_1005Metric, symbol Device:R
- added R10, R11, R12, R13, R14, R18, R5: 10k, Resistor_SMD:R_0402_1005Metric, symbol Device:R
- added R15, R16, R17, R6: R, Resistor_SMD:R_0402_1005Metric, symbol Device:R
- added R3, R4: 2k2, Resistor_SMD:R_0402_1005Metric, symbol Device:R_Small
- added R7: 220R, Resistor_SMD:R_0402_1005Metric, symbol Device:R
- added R8: 10Ω 5% 0.25W, Resistor_SMD:R_0402_1005Metric, symbol Device:R
- added R9: 33Ω 5% 0.5W, Resistor_SMD:R_0402_1005Metric, symbol Device:R
- added TP1: GND, TestPoint:TestPoint_Pad_D1.0mm, symbol Connector:TestPoint
- added TP2: 3v3, TestPoint:TestPoint_Pad_D1.0mm, symbol Connector:TestPoint
- added U1: W25Q128JVP, Package_SON:WSON-8-1EP_6x5mm_P1.27mm_EP3.4x4.3mm, symbol Memory_Flash:W25Q128JVP
- added U2: LTV-217-G, Package_SO:SOIC-4_4.55x2.6mm_P1.27mm, symbol Isolator:Optocoupler_DC_PhotoNPN_AKEC
- added U3: RythmMini, Rythm:RythmMini-v0.1, symbol Rythm:RythmMini-v0.1
- added U4: STM32H750XBHx, Package_BGA:TFBGA-265_14x14mm_Layout17x17_P0.8mm, symbol MCU_ST_STM32H7:STM32H750XBHx
- added Y1: Crystal_GND24, Crystal:Crystal_SMD_Abracon_ABM10-4Pin_2.5x2.0mm, symbol Device:Crystal_GND24
Connections:
- net GND: now also C1.2, C16.2, C17.2, C18.2, C19.2, C2.2, C23.1, C25.1, C28.2, C29.2, C3.2, C30.2, C31.2, C32.2, C33.2, C4.2, C46.1, C47.1, C48.2, C5.2, C50.2, C51.2, C52.2, C54.2, C55.2, C56.2, C57.2, C58.2, C6.2, C60.2, C61.2, C62.2, C63.2, C64.2, C67.2, C68.2, C69.2, D1.1 (K), D2.1 (K), D4.1 (K), IC1.12 (VSSD), IC1.18 (MODE), IC1.24 (VSSSPK), IC1.28 (VSSA), IC1.33 (EP), IC2.A3 (VSS), IC2.B3 (VSSQ), IC2.B8 (VSSQ), IC2.C1 (VSSQ), IC2.D1 (VSSQ), IC2.E9 (VSSQ), IC2.F1 (VSS), IC2.L3 (VSS), IC2.L9 (VSSQ), IC2.M1 (VSSQ), IC2.N1 (VSSQ), IC2.P3 (VSSQ), IC2.P8 (VSSQ), IC2.R3 (VSS), Q1.2 (S), TP1.1, U1.4 (GND), U1.9 (EP), U2.3, U4.A1 (VSS), U4.A17 (VSS), U4.B2 (VSS), U4.B6 (VSS), U4.C10 (VSS), U4.C13 (VSS), U4.C16 (VSS), U4.F1 (VSS), U4.F2 (VSS), U4.G10 (VSS), U4.G11 (VSS), U4.G16 (VSS), U4.G2 (VSS), U4.G7 (VSS), U4.G8 (VSS), U4.G9 (VSS), U4.H10 (VSS), U4.H11 (VSS), U4.H7 (VSS), U4.H8 (VSS), U4.H9 (VSS), U4.J10 (VSS), U4.J11 (VSS), U4.J16 (VSS), U4.J17 (VSS), U4.J3 (VSS), U4.J7 (VSS), U4.J8 (VSS), U4.J9 (VSS), U4.K10 (VSS), U4.K11 (VSS), U4.K15 (VSS), U4.K7 (VSS), U4.K8 (VSS), U4.K9 (VSS), U4.L10 (VSS), U4.L11 (VSS), U4.L15 (VSS), U4.L7 (VSS), U4.L8 (VSS), U4.L9 (VSS), U4.M15 (VSS), U4.N16 (VSS), U4.P1 (VSSA), U4.R4 (VSS), U4.R8 (VSS), U4.T12 (VSS), U4.U1 (VSS), U4.U17 (VSS), Y1.2, Y1.4
- new net: D1.2 (A), R16.2
- new net: D2.2 (A), R15.2
- new net: C2.1, U4.D17 (VCAP)
- new net: FB5.1, R9.1
- new net: C27.1, IC1.19 (LAUXIN)
- new net: FB4.1, R8.2
- new net: D4.2 (A), R17.2
- new net: C20.1, IC1.22 (AUXOUT2)
- new net: C29.1, IC1.27 (VREF)
- new net: C28.1, IC1.32 (MICBIAS), R3.2, R4.2
- new net: C25.2, IC1.5 (RMICN)
- new net: C21.1, IC1.21 (AUXOUT1)
- new net: FB2.2, R7.1
- new net: D3.1 (K), R7.2, U2.1
- new net: C47.2, U4.J1 (PH1), Y1.1
- new net: C46.2, U4.J2 (PH0), Y1.3
- new net: U4.E1 (NC), U4.L16 (NC)
- new net: C3.1, U4.A7 (VCAP)
- new net: C15.1, U4.M1 (VREF+)
- new net: C15.2, U4.N1 (VREF-)
- new net: C1.1, U4.U11 (VCAP)
- new net: U3.A1 (NC), U3.A9 (NC), U3.Y1 (NC), U3.Y9 (NC)
- new net: D3.2 (A), FB3.2, U2.2
- new net: C26.1, IC1.20 (RAUXIN)
- new net: IC2.E3 (NC), IC2.E7 (NC), IC2.H7 (NC), IC2.K2 (NC), IC2.K3 (NC)
- new net: C22.2, IC1.1 (LMICP)
- new net: C23.2, IC1.2 (LMICN)
- new net: C24.2, IC1.4 (RMICP)
- new net +3.3V: C16.1, C17.1, C18.1, C19.1, C32.1, C4.1, C48.1, C5.1, C50.1, C51.1, C52.1, C54.1, C55.1, C56.1, C57.1, C58.1, C6.1, C60.1, C61.1, C62.1, C63.1, C64.1, C67.1, C68.1, C69.1, F1.1, FB1.2, IC1.13 (VDDC), IC1.14 (VDDB), IC1.26 (VDDSPK), IC1.31 (VDDA), IC2.A7 (VDD), IC2.B2 (VDDQ), IC2.B7 (VDDQ), IC2.C9 (VDDQ), IC2.D9 (VDDQ), IC2.E1 (VDDQ), IC2.F9 (VDD), IC2.L1 (VDDQ), IC2.L7 (VDD), IC2.M9 (VDDQ), IC2.N9 (VDDQ), IC2.P2 (VDDQ), IC2.P7 (VDDQ), IC2.R7 (VDD), R1.1, R10.1, R11.1, R12.1, R13.1, R14.1, R16.1, R18.1, R2.1, R5.1, R6.1, R9.2, U1.8 (VCC), U4.E11 (VDD), U4.E6 (VDD), U4.E7 (PDR_ON), U4.E9 (VDD), U4.F17 (VDD33_USB), U4.F5 (VDD), U4.G13 (VDD), U4.G17 (VDD50_USB), U4.G5 (VDD), U4.H13 (VDD), U4.H5 (VDD), U4.J13 (VDD), U4.K13 (VDD), U4.K5 (VDD), U4.L13 (VDD), U4.L5 (VDD), U4.M13 (VDD), U4.M5 (VDD), U4.N10 (VDD), U4.N11 (VDD), U4.N12 (VDD), U4.N7 (VDD), U4.N8 (VDD), U4.P17 (VDD)
- new net +3.3VA: C30.1, C31.1, FB1.1, U4.L1 (VDDA)
- new net 3v3+: F1.2, Q1.1 (G), TP2.1, U3.T9 (3.3v)
- new net 3v3_GND: Q1.3 (D), U3.R9 (GND)
- new net AUX_IN_L: C27.2, U3.E9 (AUX_IN_R)
- new net AUX_IN_R: C26.2, U3.D9 (AUX_IN_L)
- new net AUX_OUT_L: C20.2, U3.B9 (AUX_OUT_L)
- new net AUX_OUT_R: C21.2, U3.C9 (AUX_OUT_R)
- new net BOOT0: R18.2, U4.E8 (BOOT0)
- new net DIN_IN_SINK: FB3.1
- new net DIN_IN_SOURCE: FB2.1
- new net DIN_MIDI_RX: R6.2, U2.4, U4.P12 (PB11)
- new net DIN_MIDI_TX: R8.1, U4.P11 (PB10)
- new net DIN_OUT_SINK: FB4.2
- new net DIN_OUT_SOURCE: FB5.2
- new net FMC_A0: IC2.G8 (A0), U4.G4 (PF0)
- new net FMC_A1: IC2.G9 (A1), U4.G3 (PF1)
- new net FMC_A10: IC2.G7 (A10), U4.T8 (PG0)
- new net FMC_A11: IC2.H9 (A11), U4.U8 (PG1)
- new net FMC_A12: IC2.H3 (A12), U4.H16 (PG2)
- new net FMC_A2: IC2.F7 (A2), U4.G1 (PF2)
- new net FMC_A3: IC2.F3 (A3), U4.H4 (PF3)
- new net FMC_A4: IC2.G1 (A4), U4.J5 (PF4)
- new net FMC_A5: IC2.G2 (A5), U4.J4 (PF5)
- new net FMC_A6: IC2.G3 (A6), U4.R7 (PF12)
- new net FMC_A7: IC2.H1 (A7), U4.P7 (PF13)
- new net FMC_A8: IC2.H2 (A8), U4.P8 (PF14)
- new net FMC_A9: IC2.J3 (A9), U4.R9 (PF15)
- new net FMC_BA0: IC2.J7 (BA0), U4.H14 (PG4)
- new net FMC_BA1: IC2.H8 (BA1), U4.G14 (PG5)
- new net FMC_CLK: IC2.J1 (CLK), U4.B12 (PD3)
- new net FMC_D0: IC2.N7 (DQ1), U4.P16 (PD14)
- new net FMC_D1: IC2.R8 (DQ0), U4.P15 (PD15)
- new net FMC_D10: IC2.M2 (DQ10), U4.T10 (PE13)
- new net FMC_D11: IC2.N2 (DQ12), U4.U10 (PE14)
- new net FMC_D12: IC2.P1 (DQ11), U4.R11 (PE15)
- new net FMC_D13: IC2.R1 (DQ13), U4.U16 (PD8)
- new net FMC_D14: IC2.N3 (DQ14), U4.T17 (PD9)
- new net FMC_D15: IC2.R2 (DQ15), U4.T16 (PD10)
- new net FMC_D16: IC2.E8 (DQ16), U4.T13 (PH8)
- new net FMC_D17: IC2.D7 (DQ17), U4.R13 (PH9)
- new net FMC_D18: IC2.D8 (DQ18), U4.P13 (PH10)
- new net FMC_D19: IC2.B9 (DQ19), U4.P14 (PH11)
- new net FMC_D2: IC2.P9 (DQ4), U4.D13 (PD0)
- new net FMC_D20: IC2.C8 (DQ20), U4.R14 (PH12)
- new net FMC_D21: IC2.A8 (DQ23), U4.D16 (PH13)
- new net FMC_D22: IC2.C7 (DQ22), U4.B17 (PH14)
- new net FMC_D23: IC2.A9 (DQ21), U4.B16 (PH15)
- new net FMC_D24: IC2.A1 (DQ26), U4.A16 (PI0)
- new net FMC_D25: IC2.B1 (DQ28), U4.A15 (PI1)
- new net FMC_D26: IC2.A2 (DQ24), U4.B15 (PI2)
- new net FMC_D27: IC2.C2 (DQ27), U4.C14 (PI3)
- new net FMC_D28: IC2.D2 (DQ29), U4.A2 (PI6)
- new net FMC_D29: IC2.C3 (DQ25), U4.B3 (PI7)
- new net FMC_D3: IC2.N8 (DQ3), U4.E12 (PD1)
- new net FMC_D30: IC2.E2 (DQ31), U4.E2 (PI9)
- new net FMC_D31: IC2.D3 (DQ30), U4.F3 (PI10)
- new net FMC_D4: IC2.R9 (DQ2), U4.U9 (PE7)
- new net FMC_D5: IC2.M8 (DQ5), U4.T9 (PE8)
- new net FMC_D6: IC2.M7 (DQ6), U4.P9 (PE9)
- new net FMC_D7: IC2.L8 (DQ7), U4.N9 (PE10)
- new net FMC_D8: IC2.L2 (DQ8), U4.P10 (PE11)
- new net FMC_D9: IC2.M3 (DQ9), U4.R10 (PE12)
- new net FMC_NBL0: IC2.K9 (DQM0), U4.C4 (PE0)
- new net FMC_NBL1: IC2.K1 (DQM1), U4.B4 (PE1)
- new net FMC_NBL2: IC2.F8 (DQM2), U4.A4 (PI4)
- new net FMC_NBL3: IC2.F2 (DQM3), U4.A3 (PI5)
- new net FMC_NE1: IC2.J8 (~{CS}), U4.F13 (PC7)
- new net FMC_SDCKE0: IC2.J2 (CKE), U4.N2 (PH2)
- new net FMC_SDNCAS: IC2.K7 (~{CAS}), U4.D6 (PG15)
- new net FMC_SDNRAS: IC2.J9 (~{RAS}), U4.T7 (PF11)
- new net FMC_SDNWE: IC2.K8 (~{WE}), U4.P4 (PH5)
- new net HPL: IC1.30 (LHP), U3.A6 (HPL)
- new net HPR: IC1.29 (RHP), U3.A7 (HPR)
- new net I2C_SCL: IC1.16 (SCLK), R1.2, U3.C1 (PB7/SCL), U4.D5 (PB8)
- new net I2C_SDA: IC1.17 (SDIO), R2.2, U3.B1 (PB8/SDA), U4.C5 (PB7)
- new net LED_STATUS: R15.1, U4.F14 (PC6)
- new net LED_STATUS2: R17.1, U4.D14 (PA10)
- new net LIN: IC1.3 (LLIN/GPIO2), U3.A2 (IN_L)
- new net MICL: C22.1, R4.1, U3.A4 (MICL)
- new net MICR: C24.1, R3.1, U3.A5 (MICR)
- new net PA11/4RX: U3.H8 (PA11/RX), U4.E17 (PA11)
- new net PA12/4TX: U3.G8 (PA12/TX), U4.E16 (PA12)
- new net PA2: U4.N3 (PA2)
- new net PA3: U4.U2 (PA3)
- new net PA5: U3.M1 (PA5/SCK), U4.T3 (PA5)
- new net PA6: U3.N1 (PA6/MISO), U4.R3 (PA6)
- new net PA7: U3.O1 (PA7/MOSI), U4.R5 (PA7)
- new net PB13: U3.Q9 (PB13), U4.U14 (PB13)
- new net PB4: U4.B7 (PB4)
- new net PB5: U3.E1 (PB5/RX), U4.A5 (PB5)
- new net PB6: U3.D1 (PB6/TX), U4.B5 (PB6)
- new net PB9: U4.D4 (PB9)
- new net QSPI_CLK: U1.6 (CLK), U4.L3 (PF10)
- new net QSPI_IO0: U1.5 (DI/IO_{0}), U4.K4 (PF8)
- new net QSPI_IO1: U1.2 (DO/IO_{1}), U4.L4 (PF9)
- new net QSPI_IO2: U1.3 (~{WP}/IO_{2}), U4.K3 (PF7)
- new net QSPI_IO3: U1.7 (~{HOLD}/~{RESET}/IO_{3}), U4.K2 (PF6)
- new net QSPI_NCS: U1.1 (~{CS}), U4.G15 (PG6)
- new net RIN: IC1.6 (RLIN/GPIO3), U3.A3 (IN_R)
- new net RST: C33.1, R5.2, U3.G1 (RESET), U4.K1 (NRST)
- new net SAI1_FS: IC1.7 (FS), U4.D2 (PE4)
- new net SAI1_MCLK: IC1.11 (MCLK), U4.C3 (PE2)
- new net SAI1_SCK: IC1.8 (BCLK), U4.D1 (PE5)
- new net SAI1_SD_A: IC1.10 (DACIN), U4.E5 (PE6)
- new net SAI1_SD_B: IC1.9 (ADCOUT), U4.D3 (PE3)
- new net SDMMC1_CK: U3.G9 (SDMMC_CLK), U4.C12 (PC12)
- new net SDMMC1_CMD: R10.2, U3.F9 (SDMMC_CMD), U4.D12 (PD2)
- new net SDMMC1_D0: R11.2, U3.K9 (SDMMC_D0), U4.E13 (PC8)
- new net SDMMC1_D1: R12.2, U3.J9 (SDMMC_D1), U4.E14 (PC9)
- new net SDMMC1_D2: R13.2, U3.I9 (SDMMC_D2), U4.A13 (PC10)
- new net SDMMC1_D3: R14.2, U3.H9 (SDMMC_D3), U4.B13 (PC11)
- new net SPKL: IC1.25 (LSPKOUT), U3.A8 (SPKL)
- new net SPKR: IC1.23 (RSPKOUT), U3.A9 (NC)
- new net SWD_CLK: U3.D8 (CLK), U4.B14 (PA14)
- new net SWD_IO: U3.E8 (IO), U4.C15 (PA13)
- new net SWD_SWO: U3.C8 (SWO), U4.C6 (PB3)
- new net USB_D+: U3.O9 (D+), U4.T15 (PB15)
- new net USB_D-: U3.P9 (D-), U4.U15 (PB14)
- new net VBAT: U3.F1 (VBAT), U4.B1 (VBAT)
- no-connect marks 0 -> 1
Other:
- note added: "MIDI DIN"
- note added: "Reverse voltage protection circuit"
- note added: "TODO: should BOOT be high or low?"
