File: hardware/boards/mini/v0.2/rythm_mini_v0.2.kicad_sch (KiCad schematic)
At the start: 99 parts, among them IC1 NAU88C22YG, IC3 IS42S16160J-6BLI, J2 Top, J3 Bottom, Q1 PMV37EN22, U1 W25Q128JVP, U2 LTV-217-G, U4 STM32H750XBHx, Y1 Crystal_GND24, Y3 32.768kHz

Commit message: mini: layout adjustments after component package changes
Parts:
- C10, C11, C12, C13, C14, C33, C48, C5, C50, C51, C52, C54, C55, C56, C57, C58, C60, C61, C62, C63, C64, C67, C68, C7, C8, C9: Digikey 1276-CL05B104KP5VPNCCT-ND -> (none); JLC C1525 -> (none)
- C16, C17, C18, C19, C28, C29, C36, C37, C38: Digikey 1276-1482-1-ND -> (none); JLC C23733 -> (none)
- C20, C21, C22, C23, C24, C25, C26, C27, C31, C32, C6: Digikey 1276-1043-1-ND -> (none); JLC C52923 -> (none)
- C30: Digikey 399-C0402C103K4REC7411CT-ND -> (none); JLC C15195 -> (none)
- C34, C35, C69: Digikey 1276-1450-1-ND -> (none); JLC C15525 -> (none)
- D1: JLC C2286 -> (none)
- D2, D4: JLC C89811 -> (none)
- D3: JLC C2128 -> (none)
- FB1: Digikey 490-5203-1-ND -> (none)
- FB2, FB3, FB4, FB5: Digikey 490-5442-1-ND -> (none)
- IC1: Digikey NAU88C22YG-ND -> (none); JLC C914209 -> (none)
- IC3: Digikey 1450-1249-ND -> (none); JLC C1351289 -> (none)
- J2, J3: Digikey H11628CT-ND -> (none); JLC C424647 -> (none)
- Q1: Digikey 1727-2306-1-ND -> (none); JLC C478164 -> (none)
- R1, R2: Digikey 311-4.7KJRCT-ND -> (none); JLC C25900 -> (none)
- R10, R11, R12, R13, R14, R18, R5: Digikey 311-10KJRCT-ND -> (none); JLC C25744 -> (none)
- R3, R4: Digikey RMCF0402FT2K20CT-ND -> (none); JLC C25879 -> (none)
- R7: Digikey A130044CT-ND -> (none); JLC C25091 -> (none)
- U1: Digikey 256-W25Q128JVPIQ-TUBE-ND -> (none); JLC C190862 -> (none)
- U2: Digikey 160-2218-1-ND -> (none); JLC C17407902 -> (none)
- U4: Digikey 497-18111-ND -> (none); JLC C405932 -> (none)
- Y3: Digikey SER4103CT-ND -> (none); JLC C32346 -> (none)
